File: board/pool/analog.kicad_sch (KiCad schematic)
At the start: 28 parts, among them J1 -0.3, J2 ORP, U1 TLV2372, U2 TLV2372, U3 TLV75801PDBV, U4 ADS1015IDGS

Commit message: Added rev 1.1 of the board
Parts:
- added C13: 100n, Capacitor_SMD:C_0805_2012Metric_Pad1.18x1.45mm_HandSolder, symbol Device:C
- added C14: 10u, Capacitor_SMD:C_0805_2012Metric_Pad1.18x1.45mm_HandSolder, symbol Device:C
- added TP8: GNDA, TestPoint:TestPoint_Pad_2.0x2.0mm, symbol Connector:TestPoint
- added U8: TEA1-0505, Converter_DCDC:Converter_DCDC_TRACO_TEA1-xxxx_THT, symbol Converter_DCDC:TEA1-0505
- TP7: value TestPoint -> GNDA
Connections:
- net +5V: now also U8.2 (+Vin); no longer C7.1, U3.1 (IN), U3.3 (EN)
- net GND: now also U8.1 (-Vin); no longer C10.2, C11.2, C7.2, C8.1, C9.2, R10.1, R12.1, U1.4 (V-), U2.4 (V-), U3.2 (GND), U4.1 (ADDR), U4.3 (GND)
- net VDDA: now also C13.1
- new net +5VA: C14.1, C7.1, U3.1 (IN), U3.3 (EN), U8.4 (+Vout)
- new net GNDA: C10.2, C11.2, C13.2, C14.2, C7.2, C8.1, C9.2, R10.1, R12.1, TP8.1, U1.4 (V-), U2.4 (V-), U3.2 (GND), U4.1 (ADDR), U4.3 (GND), U8.3 (-Vout)
Other:
- moved on the sheet: C11, C7, C8, R10, R11, R12, R9, TP7, U3
