File: board/pool/digital.kicad_sch (KiCad schematic)
At the start: 26 parts, among them J4 Raspberry_Pi_4, J5 Screw_Terminal_01x04, U5 MAX481E, U6 AP62300WU, U7 ISO1541

Commit message: Added rev 1.1 of the board
Parts:
- removed R18: 0, Resistor_SMD:R_0805_2012Metric_Pad1.20x1.40mm_HandSolder, symbol Device:R
- removed TP8: GND, TestPoint:TestPoint_THTPad_1.5x1.5mm_Drill0.7mm, symbol Connector:TestPoint
- added D1: LED, LED_THT:LED_D1.8mm_W3.3mm_H2.4mm, symbol Device:LED
- added R13: 13k, Resistor_SMD:R_0805_2012Metric_Pad1.20x1.40mm_HandSolder, symbol Device:R
- added SW1: SW_Slide_DPDT, mylib:CL-SB-22A, symbol Switch:SW_Slide_DPDT
- TP1: footprint TestPoint:TestPoint_THTPad_1.5x1.5mm_Drill0.7mm -> TestPoint:TestPoint_Pad_2.0x2.0mm
- U6: footprint Package_TO_SOT_SMD:TSOT-23-6_HandSoldering -> Package_TO_SOT_SMD:TSOT-23-6
Connections:
- net RDY_A is gone; now on net RDY: R17.2
- net +5V: no longer TP1.1, U5.8 (VCC)
- net GND: now also TP1.1, R13.1, SW1.4 (A); no longer U7.5 (GND2)
- net +3V3: now reaches C12.1, J4.1 (3V3), J4.17 (3V3), U7.1 (VCC1)
- net +3V3: now also U5.8 (VCC)
- net at J4.40 (GPIO21/SPI1_SCLK/PCM_DOUT): now also D1.2 (A)
- net at R2.1, U6.5 (EN): now also SW1.5 (B); no longer R1.2
- new net: R1.2, SW1.6 (C)
- new net: D1.1 (K), R13.2
- new net GNDA: U7.5 (GND2)
- no-connect marks 0 -> 3
Other:
- moved on the sheet: C1, J5, R1, U5
